Commit message: change obj -> stl to clarify the scene coords

File: LeapProject/Assets/urdf/robot.urdf (robot description, URDF)
Before this commit: robot leap_hand, 19 links, 18 joints
Links:
- link dip: geometry collision mesh filename=package://meshes/dip.stl; visual mesh filename=package://meshes/dip.stl
- link dip_2: geometry collision mesh filename=package://meshes/dip.stl; visual mesh filename=package://meshes/dip.stl
- link dip_3: geometry collision mesh filename=package://meshes/dip.stl; visual mesh filename=package://meshes/dip.stl
- link fingertip: geometry collision mesh filename=package://meshes/fingertip.stl; visual mesh filename=package://meshes/fingertip.stl
- link fingertip_2: geometry collision mesh filename=package://meshes/fingertip.stl; visual mesh filename=package://meshes/fingertip.stl
- link fingertip_3: geometry collision mesh filename=package://meshes/fingertip.stl; visual mesh filename=package://meshes/fingertip.stl
- link mcp_joint: geometry collision mesh filename=package://meshes/mcp_joint.stl; visual mesh filename=package://meshes/mcp_joint.stl
- link mcp_joint_2: geometry collision mesh filename=package://meshes/mcp_joint.stl; visual mesh filename=package://meshes/mcp_joint.stl
- link mcp_joint_3: geometry collision mesh filename=package://meshes/mcp_joint.stl; visual mesh filename=package://meshes/mcp_joint.stl
- link mount: geometry collision mesh filename=package://meshes/leap_mount.stl; visual mesh filename=package://meshes/leap_mount.stl
- link palm_lower: geometry collision mesh filename=package://meshes/palm_lower.stl; visual mesh filename=package://meshes/palm_lower.stl
- link pip: geometry collision mesh filename=package://meshes/pip.stl; visual mesh filename=package://meshes/pip.stl
- link pip_2: geometry collision mesh filename=package://meshes/pip.stl; visual mesh filename=package://meshes/pip.stl
- link pip_3: geometry collision mesh filename=package://meshes/pip.stl; visual mesh filename=package://meshes/pip.stl
- link pip_4: geometry collision mesh filename=package://meshes/pip.stl; visual mesh filename=package://meshes/pip.stl
- link thumb_dip: geometry collision mesh filename=package://meshes/thumb_dip.stl; visual mesh filename=package://meshes/thumb_dip.stl
- link thumb_fingertip: geometry collision mesh filename=package://meshes/thumb_fingertip.stl; visual mesh filename=package://meshes/thumb_fingertip.stl
- link thumb_pip: geometry collision mesh filename=package://meshes/thumb_pip.stl; visual mesh filename=package://meshes/thumb_pip.stl

Commit message: fixed Blender meshes with color

File: LeapProject/Assets/urdf/robot.urdf (robot description, URDF)
Before this commit: robot leap_hand, 19 links, 18 joints
Links:
- link dip: geometry collision mesh filename=package://meshes/dip.stl; visual mesh filename=package://meshes/dip_fixed.obj
- link dip_2: geometry collision mesh filename=package://meshes/dip.stl; visual mesh filename=package://meshes/dip_fixed.obj
- link dip_3: geometry collision mesh filename=package://meshes/dip.stl; visual mesh filename=package://meshes/dip_fixed.obj
- link fingertip: geometry collision mesh filename=package://meshes/fingertip.stl; visual mesh filename=package://meshes/fingertip_fixed.obj
- link fingertip_2: geometry collision mesh filename=package://meshes/fingertip.stl; visual mesh filename=package://meshes/fingertip_fixed.obj
- link fingertip_3: geometry collision mesh filename=package://meshes/fingertip.stl; visual mesh filename=package://meshes/fingertip_fixed.obj
- link mcp_joint: geometry collision mesh filename=package://meshes/mcp_joint.stl; visual mesh filename=package://meshes/mcp_joint_fixed.obj
- link mcp_joint_2: geometry collision mesh filename=package://meshes/mcp_joint.stl; visual mesh filename=package://meshes/mcp_joint_fixed.obj
- link mcp_joint_3: geometry collision mesh filename=package://meshes/mcp_joint.stl; visual mesh filename=package://meshes/mcp_joint_fixed.obj
- link mount: geometry collision mesh filename=package://meshes/leap_mount.stl; visual mesh filename=package://meshes/leap_mount_fixed.obj
- link palm_lower: geometry collision mesh filename=package://meshes/palm_lower.stl; visual mesh filename=package://meshes/palm_lower_fixed.obj
- link pip: geometry collision mesh filename=package://meshes/pip.stl; visual mesh filename=package://meshes/pip_fixed.obj
- link pip_2: geometry collision mesh filename=package://meshes/pip.stl; visual mesh filename=package://meshes/pip_fixed.obj
- link pip_3: geometry collision mesh filename=package://meshes/pip.stl; visual mesh filename=package://meshes/pip_fixed.obj
- link pip_4: geometry collision mesh filename=package://meshes/pip.stl; visual mesh filename=package://meshes/pip_fixed.obj
- link thumb_dip: geometry collision mesh filename=package://meshes/thumb_dip.stl; visual mesh filename=package://meshes/thumb_dip_fixed.obj
- link thumb_fingertip: geometry collision mesh filename=package://meshes/thumb_fingertip.stl; visual mesh filename=package://meshes/thumb_fingertip_fixed.obj
- link thumb_pip: geometry collision mesh filename=package://meshes/thumb_pip.stl; visual mesh filename=package://meshes/thumb_pip_fixed.obj
