Commit message: sanity check integrator example

File: scripts/warp/dummy.urdf (robot description, URDF)
Before this commit: robot toy_robot, 3 links, 2 joints
Links:
- removed link link1
- removed link link2
- removed link world
- added link arm1; visual box size=0.25 .05 .05
- added link arm2; visual box size=0.25 .05 .05
- added link base
Joints:
- removed joint joint1
- removed joint world_to_link1
- added joint interArm: type revolute, parent arm1, child arm2, origin xyz=0.25 0 0 rpy=0 0 0, axis 0 0 1

Commit message: upgrade dummy example with a toy cube

File: scripts/warp/dummy.urdf (robot description, URDF)
Before this commit: robot 2link_robot, 3 links, 1 joints
Links:
- link arm1: geometry collision box size=0.25 .05 .05; visual box size=0.25 .05 .05
- link arm2: geometry collision box size=0.25 .05 .05; visual box size=0.25 .05 .05
