Commit message: add dummy with mesh to two link collider script

File: scripts/warp/dummy_with_mesh.urdf (robot description, URDF)
Before this commit: robot 2link_robot, 3 links, 1 joints
Links:
- added link mesh; collision mesh filename=meshes/white_tip.obj; visual mesh filename=meshes/white_tip.obj
Joints:
- added joint tipJoint: type fixed, parent arm2, child mesh, origin xyz=0.125 0 0 rpy=0 0 0
